File: accel-brake-sig-converter-board/accel-brake-sig-converter-board.kicad_sch (KiCad schematic)
At the start: 0 parts

Commit message: add title, date, revision
Other:
- title: (none) -> accel-brake-sig-converter-board
Changed lines of the file:
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@@
 	(generator_version "8.0")
 	(paper "A4")
+	(title_block
+		(title "accel-brake-sig-converter-board")
+		(date "2024-08-06")
+		(rev "v1.0")
+	)
 	(sheet_instances
 		(path "/"

Commit message: create sch, add power circuit
Parts:
- added C1, C11, C2, C3, C4, C5, C6, C7, C9: 1u, ProjectEV_Capacitor:C_1608M, symbol ProjectEV_Capacitor:C_1608M
- added D1, D2, D3: PZ1AH11B-AU_R1_000A1, ProjectEV_Diode:PZ1AH11B-AU_R1_000A1, symbol ProjectEV_Diode:PZ1AH11B-AU_R1_000A1
- added D4, D5, D6, D7, D8, D9: B1911PG--20D000514U1930, ProjectEV_LED:B1911PG--20D000514U1930, symbol ProjectEV_LED:B1911PG--20D000514U1930
- added F1, F2, F3: 0ABB-1000-TM, ProjectEV_Fuse:0ABB-1000-TM, symbol ProjectEV_Fuse:0ABB-1000-TM
- added J1, J2, J3, J4, J5, J6: SM03B-PASS-TBT, ProjectEV_Connector_JST:SM03B-PASS-TBT, symbol ProjectEV_Connector_JST:SM03B-PASS-TBT
- added Q1, Q2, Q3: DMP3098LQ-7, ProjectEV_Transistor:DMP3098LQ-7, symbol ProjectEV_Transistor:DMP3098LQ-7
- added Q4, Q5, Q6: 2N7002K-AU_R1_000A2, ProjectEV_Transistor:2N7002K-AU_R1_000A2, symbol ProjectEV_Transistor:2N7002K-AU_R1_000A2
- added R1, R10, R13, R15, R2, R3: 100k, ProjectEV_Resistor:R_1608M, symbol ProjectEV_Resistor:R_1608M
- added R11, R12, R14: 100, ProjectEV_Resistor:R_1608M, symbol ProjectEV_Resistor:R_1608M
- added R4, R5, R6: 10k, ProjectEV_Resistor:R_1608M, symbol ProjectEV_Resistor:R_1608M
- added R7, R8, R9: 3.3k, ProjectEV_Resistor:R_1608M, symbol ProjectEV_Resistor:R_1608M
- added U1, U2, U3: NCV8711BMTW500TBG, ProjectEV_RegulatorLinear:NCV8711BMTW500TBG, symbol ProjectEV_RegulatorLinear:NCV8711BMTW500TBG
Connections:
- new net: D7.1 (K), Q6.3 (D)
- new net: D7.2 (A), R7.2
- new net: D3.2 (A), Q3.1 (G), R3.1
- new net: C1.1, C2.1, D3.1 (K), Q3.2 (S), R6.1, U3.6 (IN)
- new net: C5.1, C6.1, D1.1 (K), Q1.2 (S), R4.1, U1.6 (IN)
- new net: Q5.1 (G), R12.2, R13.2
- new net: D8.1 (K), Q5.3 (D)
- new net: R14.1, U3.5 (PG)
- new net: Q6.1 (G), R14.2, R15.2
- new net: C7.1, R10.1, R9.1, U1.1 (OUT)
- new net: C9.1, R13.1, R8.1, U2.1 (OUT)
- new net: D8.2 (A), R8.2
- new net: D4.2 (A), R4.2
- new net: C3.1, C4.1, D2.1 (K), Q2.2 (S), R5.1, U2.6 (IN)
- new net: C11.1, R15.1, R7.1, U3.1 (OUT)
- new net: R11.1, U1.5 (PG)
- new net: Q4.1 (G), R10.2, R11.2
- new net: F3.2, Q3.3 (D)
- new net: D2.2 (A), Q2.1 (G), R2.1
- new net: F2.2, Q2.3 (D)
- new net: R12.1, U2.5 (PG)
- new net: D1.2 (A), Q1.1 (G), R1.1
- new net: F1.2, Q1.3 (D)
- new net: D9.1 (K), Q4.3 (D)
- new net: F3.1, J3.1 (Pin_1)
- new net: D5.2 (A), R5.2
- new net: D6.2 (A), R6.2
- new net: F2.1, J2.1 (Pin_1)
- new net: D9.2 (A), R9.2
- new net: F1.1, J1.1 (Pin_1)
- new net ACCEL1_SIG_OUT: J1.3 (Pin_3)
- new net ACCEL2_SIG_OUT: J2.3 (Pin_3)
- new net BRAKE_SIG_OUT: J3.3 (Pin_3)
- new net GND1: C5.2, C6.2, C7.2, D4.1 (K), J1.2 (Pin_2), Q4.2 (S), R1.2, U1.3 (GND), U1.7 (EP)
- new net GND2: C3.2, C4.2, C9.2, D5.1 (K), J2.2 (Pin_2), Q5.2 (S), R2.2, U2.3 (GND), U2.7 (EP)
- new net GND3: C1.2, C11.2, C2.2, D6.1 (K), J3.2 (Pin_2), Q6.2 (S), R3.2, U3.3 (GND), U3.7 (EP)
- no-connect marks 0 -> 3
Other:
- note added: "Accel 1"
- note added: "Accel 2"
- note added: "Brake"

Commit message: 信号処理部追加
Parts:
- added C10: 1u, ProjectEV_Capacitor:C_1608M, symbol ProjectEV_Capacitor:C_1608M
- added C12: 0.1u, ProjectEV_Capacitor:C_1608M, symbol ProjectEV_Capacitor:C_1608M
- added C8: 1000p, ProjectEV_Capacitor:C_3216M, symbol ProjectEV_Capacitor:C_3216M
- added H1, H2, H3, H4: MountingHole_3.2mm_M3_Pad_Via, ProjectEV_Mechanical:MountingHole_3.2mm_M3_Pad_Via, symbol ProjectEV_Mechanical:MountingHole_3.2mm_M3_Pad_Via
- added R16, R17: 0, ProjectEV_Resistor:R_1608M, symbol ProjectEV_Resistor:R_1608M
- added R18: 1M, ProjectEV_Resistor:R_3216M, symbol ProjectEV_Resistor:R_3216M
- added R19, R20: 100k, ProjectEV_Resistor:R_1608M, symbol ProjectEV_Resistor:R_1608M
- added R21, R22: 10k, ProjectEV_Resistor:R_1608M, symbol ProjectEV_Resistor:R_1608M
- added U4: NCV20072DR2G, ProjectEV_Opamp:NCV20072DR2G, symbol ProjectEV_Opamp:NCV20072DR2G
Connections:
- net GND1: now also C10.2, C12.2, C8.2, R16.1, R18.2, R21.1, U4.4 (V-)
- net GND2: now also R16.2, R17.1
- net GND3: now also R17.2
- net +12V3: now reaches C1.1, C2.1, D3.1 (K), Q3.2 (S), R6.1, U3.6 (IN)
- net +12V1: now reaches C5.1, C6.1, D1.1 (K), Q1.2 (S), R4.1, U1.6 (IN)
- net +12V1: now also C10.1, C12.1, U4.8 (V+)
- net VCC1: now reaches C7.1, R10.1, R9.1, U1.1 (OUT)
- net VCC2: now reaches C9.1, R13.1, R8.1, U2.1 (OUT)
- net +12V2: now reaches C3.1, C4.1, D2.1 (K), Q2.2 (S), R5.1, U2.6 (IN)
- net VCC3: now reaches C11.1, R15.1, R7.1, U3.1 (OUT)
- net ACCEL1_SIG_OUT renamed ACCEL1_SIG_OUT_I
- net ACCEL2_SIG_OUT renamed ACCEL2_SIG_OUT_I
- net BRAKE_SIG_OUT renamed BRAKE_SIG_OUT_I
- new net: R19.2, U4.6 (-), U4.7
- new net: R21.2, R22.1, U4.2 (-)
- new net: R22.2, U4.1
- new net: R19.1, R20.2, U4.3 (+)
- new net ACCEL1_SIG_IN_V: R20.1
- new net Chassis: C8.1, H1.MP, R18.1
- no-connect marks 3 -> 6
Other:
- moved on the sheet: C1, C11, C2, C3, C4, C5, C6, C7, C9, D1, D2, D3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

Commit message: ブレーキセンサ部以外完成
Parts:
- added C13, C14, C19: 10n, ProjectEV_Capacitor:C_1608M, symbol ProjectEV_Capacitor:C_1608M
- added C15, C17: 1u, ProjectEV_Capacitor:C_1608M, symbol ProjectEV_Capacitor:C_1608M
- added C16, C18: 0.1u, ProjectEV_Capacitor:C_1608M, symbol ProjectEV_Capacitor:C_1608M
- added R23, R30: RT1206BRC07250RL, ProjectEV_Resistor:RT1206BRC07250RL, symbol ProjectEV_Resistor:RT1206BRC07250RL
- added R24, R25, R27, R29, R32, R34, R35: 100k, ProjectEV_Resistor:R_1608M, symbol ProjectEV_Resistor:R_1608M
- added R26, R28, R31, R33: 10k, ProjectEV_Resistor:R_1608M, symbol ProjectEV_Resistor:R_1608M
- added U5, U6: NCV20072DR2G, ProjectEV_Opamp:NCV20072DR2G, symbol ProjectEV_Opamp:NCV20072DR2G
Connections:
- net +12V2: now also C15.1, C16.1, U5.8 (V+)
- net +12V3: now also C17.1, C18.1, U6.8 (V+)
- net ACCEL1_SIG_IN_V: now also J4.3 (Pin_3), C13.1, R24.1
- net ACCEL1_SIG_OUT_I: now also U4.5 (+), R23.2
- net ACCEL2_SIG_IN_V: now also J5.3 (Pin_3), C14.1, R25.1, R27.1
- net ACCEL2_SIG_OUT_I: now also R30.2, U5.5 (+)
- net BRAKE_SIG_IN_V: now also J6.3 (Pin_3), C19.1, R32.1, R35.1
- net BRAKE_SIG_OUT_I: now also U6.5 (+)
- net GND1: now also J1.MP1 (MountPin), J1.MP2 (MountPin), J4.2 (Pin_2), J4.MP1 (MountPin), J4.MP2 (MountPin), C13.2, R24.2
- net GND2: now also J2.MP1 (MountPin), J2.MP2 (MountPin), J5.2 (Pin_2), J5.MP1 (MountPin), J5.MP2 (MountPin), C14.2, C15.2, C16.2, R25.2, R26.1, U5.4 (V-)
- net GND3: now also J3.MP1 (MountPin), J3.MP2 (MountPin), J6.2 (Pin_2), J6.MP1 (MountPin), J6.MP2 (MountPin), C17.2, C18.2, C19.2, R31.1, R35.2, U6.4 (V-)
- net VCC1: now also J4.1 (Pin_1)
- net VCC2: now also J5.1 (Pin_1)
- net VCC3: now also J6.1 (Pin_1)
- net at R22.2, U4.1: now also R23.1
- new net: R32.2, R34.1, U6.3 (+)
- new net: R28.2, R30.1, U5.1
- new net: R26.2, R28.1, U5.2 (-)
- new net: R27.2, R29.1, U5.3 (+)
- new net: R29.2, U5.6 (-), U5.7
- new net: R31.2, R33.1, U6.2 (-)
- new net: R33.2, U6.1
- new net: R34.2, U6.6 (-), U6.7
Other:
- note added: "2.2~3.8V"
- note added: "8.8~15.2mA"

Commit message: 回路図完成
Parts:
- added R33: RT1206BRC07250RL, ProjectEV_Resistor:RT1206BRC07250RL, symbol ProjectEV_Resistor:RT1206BRC07250RL
- F1, F2, F3: Mouser番号 (none) -> 530-0ABB-1000-TM
- renumbered C8 to C1, C11 to C10, C10 to C11, C15 to C12, C17 to C13, C12 to C14, C16 to C15, C18 to C16, C13 to C17, C14 to C18, C6 to C2, C4 to C3, C2 to C4, C3 to C6, C1 to C7, C7 to C8, D9 to D7, D7 to D9, R18 to R1, R11 to R10, R12 to R11, R14 to R12, R10 to R13, R13 to R14, R9 to R16, R8 to R17, R7 to R18, R21 to R19, R16 to R2, R26 to R21, R27 to R22, R31 to R23, R32 to R24, R22 to R25, R19 to R26, R28 to R27, R29 to R28, R33 to R29, R17 to R3, R34 to R30, R23 to R31, R30 to R32, R24 to R34, R25 to R35, R35 to R36, R1 to R4, R2 to R5, R3 to R6, R4 to R7, R5 to R8, R6 to R9
Connections:
- net BRAKE_SIG_OUT_I: now also R33.2
- net at R29.2, U6.1: now also R33.1

Commit message: update symbol
Parts:
- R1, R31, R32, R33: Package 3216 -> 3216M
- R10, R11, R12, R13, R14, R15, R16, R17, R18, R19, R2, R20, R21, R22, R23, R24, R25, R26, R27, R28, R29, R3, R30, R34, R35, R36, R4, R5, R6, R7, R8, R9: Package 1608 -> 1608M
Changed lines of the file:
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@@
 			)
 		)
-		(property "Package" "1608"
+		(property "Package" "1608M"
 			(at 69.85 157.4799 0)
 			(effects
@@
 			)
 		)
-		(property "Package" "1608"
+		(property "Package" "1608M"
 			(at 254 22.86 90)
 			(effects
@@
 			)
 		)
-		(property "Package" "3216"
+		(property "Package" "3216M"
 			(at 39.37 203.1999 0)
 			(effects
@@
 			)
 		)
-		(property "Package" "1608"
+		(property "Package" "1608M"
 			(at 238.76 149.86 90)
 			(effects
@@
 			)
 		)
-		(property "Package" "1608"
+		(property "Package" "1608M"
 			(at 53.34 213.36 90)
 			(effects
@@
 			)
 		)
-		(property "Package" "1608"
+		(property "Package" "1608M"
 			(at 162.56 160.02 90)
 			(effects
@@
 			)
 		)
-		(property "Package" "1608"
+		(property "Package" "1608M"
 			(at 179.07 96.5199 0)
 			(effects
@@
 			)
 		)
-		(property "Package" "1608"
+		(property "Package" "1608M"
 			(at 105.41 45.7199 0)
 			(effects
@@
 			)
 		)
-		(property "Package" "1608"
+		(property "Package" "1608M"
 			(at 179.07 147.3199 0)
 			(effects
@@
 			)
 		)
-		(property "Package" "1608"
+		(property "Package" "1608M"
 			(at 162.56 58.42 90)
 			(effects
@@
 			)
 		)
-		(property "Package" "3216"
+		(property "Package" "3216M"
 			(at 274.32 35.56 90)
 			(effects
@@
 			)
 		)
-		(property "Package" "1608"
+		(property "Package" "1608M"
 			(at 238.76 73.66 90)
 			(effects
@@
 			)
 		)
-		(property "Package" "1608"
+		(property "Package" "1608M"
 			(at 69.85 55.8799 0)
 			(effects
@@
 			)
 		)
-		(property "Package" "3216"
+		(property "Package" "3216M"
 			(at 274.32 137.16 90)
 			(effects
@@
 			)
 		)
-		(property "Package" "1608"
+		(property "Package" "1608M"
 			(at 69.85 106.6799 0)
 			(effects
@@
 			)
 		)
-		(property "Package" "1608"
+		(property "Package" "1608M"
 			(at 168.91 109.2199 0)
 			(effects
@@
 			)
 		)
-		(property "Package" "1608"
+		(property "Package" "1608M"
 			(at 238.76 124.46 90)
 			(effects
@@
 			)
 		)
-		(property "Package" "1608"
+		(property "Package" "1608M"
 			(at 254 124.46 90)
 			(effects
@@
 			)
 		)
-		(property "Package" "1608"
+		(property "Package" "1608M"
 			(at 372.11 50.7999 0)
 			(effects
@@
 			)
 		)
-		(property "Package" "1608"
+		(property "Package" "1608M"
 			(at 254 73.66 90)
 			(effects
@@
 			)
 		)
-		(property "Package" "1608"
+		(property "Package" "1608M"
 			(at 43.18 213.36 90)
 			(effects
@@
 			)
 		)
-		(property "Package" "3216"
+		(property "Package" "3216M"
 			(at 274.32 86.36 90)
 			(effects
@@
 			)
 		)
-		(property "Package" "1608"
+		(property "Package" "1608M"
 			(at 238.76 48.26 90)
 			(effects
@@
 			)
 		)
-		(property "Package" "1608"
+		(property "Package" "1608M"
 			(at 238.76 22.86 90)
 			(effects
@@
 			)
 		)
-		(property "Package" "1608"
+		(property "Package" "1608M"
 			(at 254 149.86 90)
 			(effects
@@
 			)
 		)
-		(property "Package" "1608"
+		(property "Package" "1608M"
 			(at 168.91 160.0199 0)
 			(effects
@@
 			)
 		)
-		(property "Package" "1608"
+		(property "Package" "1608M"
 			(at 179.07 45.7199 0)
 			(effects
@@
 			)
 		)
-		(property "Package" "1608"
+		(property "Package" "1608M"
 			(at 105.41 96.5199 0)
 			(effects
@@
 			)
 		)
-		(property "Package" "1608"
+		(property "Package" "1608M"
 			(at 105.41 147.3199 0)
 			(effects
@@
 			)
 		)
-		(property "Package" "1608"
+		(property "Package" "1608M"
 			(at 254 99.06 90)
 			(effects
@@
 			)
 		)
-		(property "Package" "1608"
+		(property "Package" "1608M"
 			(at 168.91 58.4199 0)
 			(effects
@@
 			)
 		)
-		(property "Package" "1608"
+		(property "Package" "1608M"
 			(at 238.76 99.06 90)
 			(effects
@@
 			)
 		)
-		(property "Package" "1608"
+		(property "Package" "1608M"
 			(at 162.56 109.22 90)
 			(effects
@@
 			)
 		)
-		(property "Package" "1608"
+		(property "Package" "1608M"
 			(at 372.11 101.5999 0)
 			(effects
@@
 			)
 		)
-		(property "Package" "1608"
+		(property "Package" "1608M"
 			(at 372.11 152.3999 0)
 			(effects
@@
 			)
 		)
-		(property "Package" "1608"
+		(property "Package" "1608M"
 			(at 254 48.26 90)
 			(effects
